File: pcbs/led_board/led_board.kicad_pcb (KiCad board)
At the start: 2 copper layers, 22 x 16.5 mm, 6 parts, among them J1 JST S2B-ZR, U1 BCR401UW6Q-7

Commit message: small updates and BOM
Other:
- board text removed: ".401"
Changed lines of the file:
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@@
 		)
 		(property "Value" "BCR401UW6Q-7"
-			(at 1.0087 3.516 0)
+			(at 3.238 0.016 0)
 			(unlocked yes)
-			(layer "F.Fab")
-			(effects
-				(font
-					(size 0.2 0.2)
-					(thickness 0.05)
+			(layer "Cmts.User")
+			(effects
+				(font
+					(size 0.5 0.5)
+					(thickness 0.1)
 					(bold yes)
 				)
@@
 				(font
 					(size 1.27 1.27)
-					(thickness 0.15)
-				)
-			)
-		)
-		(property "Digikey" "https://www.digikey.com/en/products/detail/diodes-incorporated/BCR401UW6Q-7/7352843"
-			(at 0 0 270)
-			(unlocked yes)
-			(layer "F.Fab")
-			(hide yes)
-			(effects
-				(font
-					(size 1 1)
 					(thickness 0.15)
 				)
@@
 			(at 0.768719 -3.16982 0)
 			(unlocked yes)
-			(layer "F.Fab")
+			(layer "Cmts.User")
 			(effects
 				(font
@@
 		(property "Value" "630NM MTE7063NK2-UR"
 			(at 1.163079 0.917784 0)
-			(layer "F.Fab")
+			(layer "Cmts.User")
 			(effects
 				(font
@@
 				(font
 					(size 1.27 1.27)
-					(thickness 0.15)
-				)
-				(justify mirror)
-			)
-		)
-		(property "Sim.Pins" "1=K 2=A"
-			(at 0 0 180)
-			(unlocked yes)
-			(layer "B.Fab")
-			(hide yes)
-			(effects
-				(font
-					(size 1 1)
 					(thickness 0.15)
 				)
@@
 		)
 	)
-	(gr_text ".401"
-		(at 149.302948 108.202566 0)
-		(layer "F.Fab")
-		(effects
-			(font
-				(size 0.373888 0.373888)
-				(thickness 0.032512)
-			)
-			(justify left bottom)
-		)
-	)
 	(gr_text "+"
 		(at 151.4989 100.7464 0)
-		(layer "F.Fab")
+		(layer "B.SilkS")
 		(effects
 			(font
@@
 	(gr_text "-"
 		(at 159 101 0)
-		(layer "F.Fab")
+		(layer "B.SilkS")
 		(effects
 			(font

Commit message: update led board to version 0.41
Parts:
- J1: value JST S2B-ZR -> CONN HEADER R/A 2POS 1.5MM; footprint footprints:JST_ZH_2POS_RA_S2B-ZR -> footprints:JST_ZH_2POS_RA
- LED1: value 630NM MTE7063NK2-UR -> 630nm 1.9V 50mA
- R1: footprint footprints:R_1206_3216Metric_Pad1.30x1.75mm_HandSolder -> footprints:R_1206
- U1: value BCR401UW6Q-7 -> 1.4-40V PWM Dimmer 100mA; footprint footprints:LED_driver_SOT-23-6_SOT95P285X140-6N -> footprints:SOT-23-6
Connections:
- R1 pad 1: Net-(U1-REXT) -> unconnected-(R1-Pad1)
- R1 pad 2: +5V -> unconnected-(R1-Pad2)
- U1 pad 6: Net-(U1-REXT) -> unconnected-(U1-REXT-Pad6)
Routing:
- net Net-(U1-REXT): track 12.7 -> 0.00 mm
- net (no net): track 0.00 -> 12.7 mm
