File: pcbs/sensor_board/sensor_board.kicad_sch (KiCad schematic)
At the start: 46 parts, among them J1 1.5mm, J2 2.5mm, J3 2.5mm, J4 1.5 mm, J5 RJ45, J6 Conn_01x06, J7 Conn_01x02, J8 Conn_01x02, Q1 220mA / 50V, Q2 220mA / 50V, Q3 220mA / 50V, U1 8-28V in / 5V 5W out, U2 8x GPIO, U3 4x PWM, U4 1 MOhm, U5 100 kOhm

Commit message: fix sensor board 1 MOhm trimpot wiring error (bumped to version 2.1)
Connections:
- net +5V: no longer U4.1 (A1)
- net at U4.2 (W1), U5.6 (W): now also U4.1 (A1)
Other:
- note added: "Note for R4: 1.4 version PCBs were retroactively upgraded to 56 kOhm, later version are back to 10 kOhm since the 1 MOhm amplifier covers the range."
- note removed: "this was 10 kOhm originally (in 1.4) but has now moved to 56 kOhm for the other LEDs (600nm and 880nm) but if we have a 1 MOhm secondary digipot in there, should go back to 10 kOhm! (so total range is 10 kOhm to 1.1 MOhm) Note: 1.4 version PCBs were retroactively upgraded to 56 kOhm"
Changed lines of the file:
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@@
 	(title_block
 		(title "${PROJ_TITLE}")
-		(date "2025-11-22")
+		(date "2026-07-07")
 		(rev "${PROJ_REV}")
 		(comment 1 "https://creativecommons.org/licenses/by-sa/4.0/")
@@
 		)
 	)
-	(text "this was 10 kOhm originally (in 1.4) but\nhas now moved to 56 kOhm for the other\nLEDs (600nm and 880nm) but if we have\na 1 MOhm secondary digipot in there, should go back\nto 10 kOhm! (so total range is 10 kOhm to 1.1 MOhm)\n\nNote: 1.4 version PCBs were retroactively upgraded\nto 56 kOhm"
+	(text "Note for R4: 1.4 version PCBs were retroactively\nupgraded to 56 kOhm, later version are back to \n10 kOhm since the 1  MOhm amplifier covers the range."
 		(exclude_from_sim no)
-		(at 209.804 267.208 0)
+		(at 239.776 259.842 0)
 		(effects
 			(font
@@
 		(color 0 0 0 0)
 	)
+	(junction
+		(at 233.68 207.01)
+		(diameter 0)
+		(color 0 0 0 0)
+	)
 	(no_connect
 		(at 193.04 204.47)
@@
 	(wire
 		(pts
-			(xy 254 179.07) (xy 254 176.53)
-		)
-		(stroke
-			(width 0)
-			(type default)
-		)
-	)
-	(wire
-		(pts
 			(xy 347.98 45.72) (xy 340.36 45.72)
 		)
@@
 	(wire
 		(pts
+			(xy 233.68 207.01) (xy 233.68 209.55)
+		)
+		(stroke
+			(width 0)
+			(type default)
+		)
+	)
+	(wire
+		(pts
 			(xy 162.56 111.76) (xy 168.91 111.76)
 		)
@@
 	)
 	(symbol
-		(lib_id "symbols:+5V")
-		(at 233.68 209.55 270)
-		(unit 1)
-		(body_style 1)
-		(exclude_from_sim no)
-		(in_bom yes)
-		(on_board yes)
-		(in_pos_files yes)
-		(dnp no)
-		(property "Reference" "#PWR045"
-			(at 229.87 209.55 0)
-			(hide yes)
-			(show_name no)
-			(do_not_autoplace no)
-			(effects
-				(font
-					(size 1.27 1.27)
-				)
-			)
-		)
-		(property "Value" "+5V"
-			(at 237.49 209.55 90)
-			(show_name no)
-			(do_not_autoplace no)
-			(effects
-				(font
-					(size 1.5 1.5)
-				)
-				(justify left)
-			)
-		)
-		(property "Footprint" ""
-			(at 233.68 209.55 0)
-			(hide yes)
-			(show_name no)
-			(do_not_autoplace no)
-			(effects
-				(font
-					(size 1.27 1.27)
-				)
-			)
-		)
-		(property "Datasheet" ""
-			(at 233.68 209.55 0)
-			(hide yes)
-			(show_name no)
-			(do_not_autoplace no)
-			(effects
-				(font
-					(size 1.27 1.27)
-				)
-			)
-		)
-		(property "Description" "Power symbol creates a global label with name \"+5V\""
-			(at 233.68 209.55 0)
-			(hide yes)
-			(show_name no)
-			(do_not_autoplace no)
-			(effects
-				(font
-					(size 1.27 1.27)
-				)
-			)
-		)
-		(pin "1"
-		)
-		(instances
-			(project "sensor_board"
-				(path "/2e363057-5f2b-4813-9b6e-20c9934d11ef"
-					(reference "#PWR045")
-					(unit 1)
-				)
-			)
-		)
-	)
-	(symbol
 		(lib_id "symbols:GND")
 		(at 184.15 165.1 270)
@@
 			)
 		)
-		(property "Datasheet" "https://www.analog.com/media/en/technical-documentation/data-sheets/AD5241_5242.pdf"
+		(property "Datasheet" "https://www.analog.com/media/en/technical-documentation/data-sheets/ad5241_ad5242.pdf"
 			(at 233.68 209.55 0)
 			(hide yes)
@@
 		)
 		(property "MPN" "AD5241BRZ1M"
-			(at 212.852 190.754 0)
+			(at 212.852 213.106 0)
 			(show_name no)
 			(do_not_autoplace yes)
